File: PCB/PiPowerHat.sch (EAGLE design)
At the start: 48 parts, among them J3 Display, J4 FAN1, K1 PIN20X2, Q1 NX2301P, U1 EEPROM24, U2 INA219AIDCNRSOIC, U3 TSL2561T, U4 DS18B20, U5 DS1820SOIC, U6 74AC125

Commit message: Added some improvements...
Parts:
- removed R5: 10k, resistor:R-EU_M0805
- added JP3: (no value), SparkFun-Connectors:M02POLAR
- added JP5: (no value), SparkFun-Connectors:M05PTH
- added SURVO-0, SURVO-1: (no value), SparkFun-Connectors:M03PTH
- J3: device SparkFun-Connectors:M04POLAR -> SparkFun-Connectors:M06POLAR
Connections:
- net ID_SD renamed ID_SDA
- removed net N$10: R5.2, U2.A1
- new net BCM10_MOSI: JP5.4, K1.19
- new net BCM11_SCLK: JP5.2, K1.23
- new net BCM14_TXD: K1.8
- new net BCM15_RXD: K1.10
- new net BCM22: K1.15
- new net BCM5: K1.29
- new net BCM8_CE0: K1.24
- new net BCM9_MISO: JP5.3, K1.21
- new net N$1: K1.18
- new net NFC_INT: J3.6, K1.13
- new net NFC_RESET: J3.5, K1.11
- new net SURVO_0: SURVO-0.2, U6G3.Q
- new net SURVO_0_PWM: K1.31, U6G3.D
- new net SURVO_1: SURVO-1.2, U6G2.Q
- new net SURVO_1_PWM: K1.32, U6G2.D
- net +3V3: now also J3.2, JP5.5
- net +5V: now also SURVO-0.3, SURVO-1.3
- net GND: now also JP3.1, JP5.1, SURVO-0.1, SURVO-1.1, U2.A1; no longer R5.1, U6G2.D, U6G3.D
- net PI_5V: now also JP3.2; no longer J3.2
Other:
- note added: "BCM 18"
- note added: "Possible extra features: 7) GPIO for NFC reader (I2C with 3v3 + reset) 8) RFID door tag reader (MakeSpace version) 9) TX/RX/3v3 connector for serial device"
- note removed: "Possible extra features: 4) On-board string of Neopixel (or other) LEDs to light the printer 6) GPIO (clk/data) for load cell (filament weight)? 7) GPIO for NFC reader (I2C + reset) 5, 6 & 7 - seperate PCB by base of printer."
- note removed: "light sensor"
- moved on the sheet: C8, U6PWR
